Commit message: 20210524

File: casus_support/urdf/casus.xacro (robot description, xacro)
@@ -13,5 +13,5 @@
     <xacro:include filename="$(find casus_support)/urdf/logical_camera/logical_camera.urdf.xacro"/>
     <xacro:logical_camera_urdf prefix="logical_camera1_" logical_camera_parent="world_interface">
-    <origin xyz="0.55 0.9 1.4" rpy="0 1.5708 0"/>
+    <origin xyz="-0.74 0.32 1.2" rpy="0 1.7 0"/>
     </xacro:logical_camera_urdf>
     <!-- Shipping Container -->
@@ -23,6 +23,27 @@
     <xacro:include filename="$(find casus_support)/urdf/shipping_container_conveyor/shipping_container_conveyor.urdf.xacro"/>
     <xacro:shipping_container_conveyor_urdf shipping_container_conveyor_prefix="conveyor1_" shipping_container_conveyor_parent="world_interface">
-    <origin xyz="0.04 -1 0.0" rpy="0 0 0"/>
+    <origin xyz="0.04 -1 0.13" rpy="0 0 0"/>
     </xacro:shipping_container_conveyor_urdf>
+    <!-- yellow_bin 1 -->
+    <xacro:include filename="$(find casus_support)/urdf/yellow_bin/yellow_bin.urdf.xacro"/>
+    <xacro:yellow_bin_urdf yellow_bin_prefix="yellow_bin1_" yellow_bin_parent="world_interface">
+    <origin xyz="-0.95 -0.49 0.95" rpy="0 -0.19 3.14"/>
+    </xacro:yellow_bin_urdf>
+    <!-- yellow_bin 2 -->
+    <xacro:yellow_bin_urdf yellow_bin_prefix="yellow_bin2_" yellow_bin_parent="world_interface">
+    <origin xyz="-0.95 0.32 0.95" rpy="0 -0.19 3.14"/>
+    </xacro:yellow_bin_urdf>
+    <!-- yellow_bin 3 -->
+    <xacro:yellow_bin_urdf yellow_bin_prefix="yellow_bin3_" yellow_bin_parent="world_interface">
+    <origin xyz="-0.95 1.13 0.95" rpy="0 -0.19 3.14"/>
+    </xacro:yellow_bin_urdf>
+    <!-- yellow_bin 4 -->
+    <xacro:yellow_bin_urdf yellow_bin_prefix="yellow_bin4_" yellow_bin_parent="world_interface">
+    <origin xyz="-0.95 1.94 0.95" rpy="0 -0.19 3.14"/>
+    </xacro:yellow_bin_urdf>
+     <!-- yellow_bin 5 -->
+    <xacro:yellow_bin_urdf yellow_bin_prefix="yellow_bin5_" yellow_bin_parent="world_interface">
+    <origin xyz="-0.95 2.75 0.95" rpy="0 -0.19 3.14"/>
+    </xacro:yellow_bin_urdf>
     <!-- Robot1 Pedestal -->
     <xacro:include filename="$(find casus_support)/urdf/robot_pedestal/robot_pedestal.urdf.xacro"/>
@@ -31,6 +52,6 @@
     </xacro:robot_pedestal_urdf>
     <!-- Robot1 -->
-    <xacro:include filename="$(find ur_description)/urdf/ur5.urdf.xacro"/>
-    <xacro:ur5_robot prefix="robot1_" joint_limited="true"/>
+    <xacro:include filename="$(find ur_description)/urdf/ur10.urdf.xacro"/>
+    <xacro:ur10_robot prefix="robot1_" joint_limited="true"/>
     <!-- Vacuum Gripper1 -->
     <xacro:include filename="$(find casus_support)/urdf/vacuum_gripper/vacuum_gripper.urdf.xacro"/>
@@ -38,5 +59,5 @@
     <!-- robot1 to pedestal. -->
     <joint name="robot1_to_pedestal" type="fixed">
-        <origin xyz="0 0 0.6" rpy="0 0 -1.57" />
+        <origin xyz="0 0 0.6" rpy="0 0 1.57" />
         <parent link="robot1_pedestal_link" />
         <child link="robot1_base_link" />

File: casus_support/urdf/shipping_container/shipping_container.urdf.xacro (robot description, xacro)
@@ -14,10 +14,10 @@
       <visual>
         <geometry>
-          <mesh filename="package://casus_gazebo/models/shipping_container_ariac/meshes/ShippingContainer_Textured.obj" scale="1 1 1"/>
+          <mesh filename="package://casus_gazebo/models/shipping_container_ariac/meshes/ShippingContainer_Textured.obj" scale="1.3 0.7 1.0"/>
         </geometry>
       </visual>
       <collision>
         <geometry>
-          <mesh filename="package://casus_gazebo/models/shipping_container_ariac/meshes/ShippingContainer_Textured.obj" scale="1 1 1"/>
+          <mesh filename="package://casus_gazebo/models/shipping_container_ariac/meshes/ShippingContainer_Textured.obj" scale="1.3 0.7 1.0"/>
         </geometry>
       </collision>

File: casus_support/urdf/shipping_container_conveyor/shipping_container_conveyor.urdf.xacro (robot description, xacro)
@@ -14,10 +14,10 @@
       <visual>
         <geometry>
-          <mesh filename="package://casus_gazebo/models/shipping_container_conveyor_ariac/meshes/ShippingContainer_Textured.obj" scale="1 1 1"/>
+          <mesh filename="package://casus_gazebo/models/shipping_container_conveyor_ariac/meshes/ShippingContainer_Textured.obj" scale="1 0.7 1.0"/>
         </geometry>
       </visual>
       <collision>
         <geometry>
-          <mesh filename="package://casus_gazebo/models/shipping_container_conveyor_ariac/meshes/ShippingContainer_Textured.obj" scale="1 1 1"/>
+          <mesh filename="package://casus_gazebo/models/shipping_container_conveyor_ariac/meshes/ShippingContainer_Textured.obj" scale="1 0.7 1.0"/>
         </geometry>
       </collision>

Commit message: 20210525

File: casus_support/urdf/casus.xacro (robot description, xacro)
@@ -13,36 +13,36 @@
     <xacro:include filename="$(find casus_support)/urdf/logical_camera/logical_camera.urdf.xacro"/>
     <xacro:logical_camera_urdf prefix="logical_camera1_" logical_camera_parent="world_interface">
-    <origin xyz="-0.74 0.32 1.2" rpy="0 1.7 0"/>
+    <origin xyz="-0.95 0.32 1.25" rpy="3.14 2 3.14"/>
     </xacro:logical_camera_urdf>
     <!-- Shipping Container -->
-    <xacro:include filename="$(find casus_support)/urdf/shipping_container/shipping_container.urdf.xacro"/>
-    <xacro:shipping_container_urdf shipping_container_prefix="container1_" shipping_container_parent="world_interface">
+    <xacro:include filename="$(find casus_support)/urdf/shipping_container_short/shipping_container_short.urdf.xacro"/>
+    <xacro:shipping_container_short_urdf shipping_container_short_prefix="container1_" shipping_container_short_parent="world_interface">
     <origin xyz="0.275 -1 0.0" rpy="0 0 0"/>
-    </xacro:shipping_container_urdf>
+    </xacro:shipping_container_short_urdf>
     <!-- shipping_container_conveyor -->
-    <xacro:include filename="$(find casus_support)/urdf/shipping_container_conveyor/shipping_container_conveyor.urdf.xacro"/>
-    <xacro:shipping_container_conveyor_urdf shipping_container_conveyor_prefix="conveyor1_" shipping_container_conveyor_parent="world_interface">
-    <origin xyz="0.04 -1 0.13" rpy="0 0 0"/>
-    </xacro:shipping_container_conveyor_urdf>
+    <xacro:include filename="$(find casus_support)/urdf/shipping_container_conveyor_tall/shipping_container_conveyor_tall.urdf.xacro"/>
+    <xacro:shipping_container_conveyor_tall_urdf shipping_container_conveyor_tall_prefix="conveyor1_" shipping_container_conveyor_tall_parent="world_interface">
+    <origin xyz="0.04 -1 0" rpy="0 0 0"/>
+    </xacro:shipping_container_conveyor_tall_urdf>
     <!-- yellow_bin 1 -->
     <xacro:include filename="$(find casus_support)/urdf/yellow_bin/yellow_bin.urdf.xacro"/>
     <xacro:yellow_bin_urdf yellow_bin_prefix="yellow_bin1_" yellow_bin_parent="world_interface">
-    <origin xyz="-0.95 -0.49 0.95" rpy="0 -0.19 3.14"/>
+    <origin xyz="-0.775 -0.49 0.75" rpy="0 -0.19 3.14"/>
     </xacro:yellow_bin_urdf>
     <!-- yellow_bin 2 -->
     <xacro:yellow_bin_urdf yellow_bin_prefix="yellow_bin2_" yellow_bin_parent="world_interface">
-    <origin xyz="-0.95 0.32 0.95" rpy="0 -0.19 3.14"/>
+    <origin xyz="-0.775 0.32 0.75" rpy="0 -0.19 3.14"/>
     </xacro:yellow_bin_urdf>
     <!-- yellow_bin 3 -->
     <xacro:yellow_bin_urdf yellow_bin_prefix="yellow_bin3_" yellow_bin_parent="world_interface">
-    <origin xyz="-0.95 1.13 0.95" rpy="0 -0.19 3.14"/>
+    <origin xyz="-0.775 1.13 0.75" rpy="0 -0.19 3.14"/>
     </xacro:yellow_bin_urdf>
     <!-- yellow_bin 4 -->
     <xacro:yellow_bin_urdf yellow_bin_prefix="yellow_bin4_" yellow_bin_parent="world_interface">
-    <origin xyz="-0.95 1.94 0.95" rpy="0 -0.19 3.14"/>
+    <origin xyz="-0.775 1.94 0.75" rpy="0 -0.19 3.14"/>
     </xacro:yellow_bin_urdf>
      <!-- yellow_bin 5 -->
     <xacro:yellow_bin_urdf yellow_bin_prefix="yellow_bin5_" yellow_bin_parent="world_interface">
-    <origin xyz="-0.95 2.75 0.95" rpy="0 -0.19 3.14"/>
+    <origin xyz="-0.775 2.75 0.75" rpy="0 -0.19 3.14"/>
     </xacro:yellow_bin_urdf>
     <!-- Robot1 Pedestal -->

File: casus_support/urdf/shipping_container/shipping_container.xacro (robot description, xacro)
@@ -11,9 +11,9 @@
   <link name="world_interface" />
   <!-- URDF -->
-  <xacro:include filename="$(find casus_support)/urdf/shipping_container_mobile/shipping_container.urdf.xacro"/>
+  <xacro:include filename="$(find casus_support)/urdf/shipping_container/shipping_container.urdf.xacro"/>
   <xacro:shipping_container_urdf shipping_container_prefix="$(arg shipping_container_prefix)" shipping_container_parent="$(arg shipping_container_parent)">
      <origin xyz="$(arg x) $(arg y) $(arg z)" rpy="$(arg R) $(arg P) $(arg Y)"/>
   </xacro:shipping_container_urdf>
   <!-- Gazebo -->
-  <xacro:include filename="$(find casus_support)/urdf/shipping_container_mobile/shipping_container.gazebo.xacro"/>
+  <xacro:include filename="$(find casus_support)/urdf/shipping_container/shipping_container.gazebo.xacro"/>
 </robot>

File: casus_support/urdf/shipping_container_conveyor/shipping_container_conveyor.xacro (robot description, xacro)
@@ -11,9 +11,9 @@
   <link name="world_interface" />
   <!-- URDF -->
-  <xacro:include filename="$(find casus_support)/urdf/shipping_container_conveyor_mobile/shipping_container_conveyor.urdf.xacro"/>
+  <xacro:include filename="$(find casus_support)/urdf/shipping_container_conveyor/shipping_container_conveyor.urdf.xacro"/>
   <xacro:shipping_container_conveyor_urdf shipping_container_conveyor_prefix="$(arg shipping_container_conveyor_prefix)" shipping_container_conveyor_parent="$(arg shipping_container_conveyor_parent)">
      <origin xyz="$(arg x) $(arg y) $(arg z)" rpy="$(arg R) $(arg P) $(arg Y)"/>
   </xacro:shipping_container_conveyor_urdf>
   <!-- Gazebo -->
-  <xacro:include filename="$(find casus_support)/urdf/shipping_container_conveyor_mobile/shipping_container_conveyor.gazebo.xacro"/>
+  <xacro:include filename="$(find casus_support)/urdf/shipping_container_conveyor/shipping_container_conveyor.gazebo.xacro"/>
 </robot>
